Commit message: calibration

File: src/scout_unitree/urdf/robot.xacro (robot description, xacro)
@@ -5,8 +5,7 @@
     <xacro:include filename="$(find z1_description)/xacro/transmission.xacro" />
     <xacro:arg name="UnitreeGripper" default="false" />
-    <link name="world" />
     <joint name="base_static_joint" type="fixed">
-        <origin rpy="0 0 0" xyz="0 0 0" />
-        <parent link="world" />
+        <origin rpy="0 0 0" xyz="0.1082 0 0.368" />
+        <parent link="base_link" />
         <child link="link00" />
     </joint>
