Commit message: None

File: src/scout_unitree/scout_unitree_gazebo/urdf/connections.urdf (robot description, URDF)
Before this commit: robot connect_slabs, 4 links, 4 joints
Links:
- link slab01_link: geometry collision mesh filename=package://scout_unitree_gazebo/meshes/2mm_slab.STL scale=0.001 0.001 0.001; visual mesh filename=package://scout_unitree_gazebo/meshes/2mm_slab.STL scale=0.001 0.001 0.001
- link slab02_link: geometry collision mesh filename=package://scout_unitree_gazebo/meshes/7mm_slab.STL scale=0.001 0.001 0.001; visual mesh filename=package://scout_unitree_gazebo/meshes/7mm_slab.STL scale=0.001 0.001 0.001
- link slab03_link: geometry collision mesh filename=package://scout_unitree_gazebo/meshes/lidar_camera_connecti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 scale=0.001 0.001 0.001; visual mesh filename=package://scout_unitree_gazebo/meshes/lidar_camera_connecti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 scale=0.001 0.001 0.001
- link slab04_link: geometry collision mesh filename=package://scout_unitree_gazebo/meshes/lv_frame.STL scale=0.001 0.001 0.001; visual mesh filename=package://scout_unitree_gazebo/meshes/lv_frame.STL scale=0.001 0.001 0.001
